File: Nomad/Nomad.kicad_sch (KiCad schematic)
At the start: 52 parts, among them J1 Barrel_Jack, U1 ESP32-DEVKITC-32UE, U2 BU18SD5WG-TL, U3 BU33SD5WG-TR, U4 XL1509-5.0, U5 PTAS2780RYAR

Commit message: retouches schema elec
Other:
- note added: "1.0"
- note added: "Projet S7 "Nomad""
Changed lines of the file:
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@@
 	(generator_version "9.0")
 	(paper "A4")
+	(text "Projet S7 \"Nomad\""
+		(exclude_from_sim no)
+		(at 186.182 189.738 0)
+		(effects
+			(font
+				(size 1.905 1.905)
+				(thickness 0.2381)
+				(color 0 0 0 1)
+			)
+			(justify left)
+		)
+	)
+	(text "1.0"
+		(exclude_from_sim no)
+		(at 269.748 193.548 0)
+		(effects
+			(font
+				(size 1.27 1.27)
+			)
+			(justify left)
+		)
+	)
 	(text_box "Amplificateur audio"
 		(exclude_from_sim no)
@@
 	)
 	(junction
+		(at 46.99 35.56)
+		(diameter 0)
+		(color 0 0 0 0)
+	)
+	(junction
 		(at 247.65 116.84)
 		(diameter 0)
@@
 		(color 0 0 0 0)
 	)
-	(junction
-		(at 36.83 35.56)
-		(diameter 0)
-		(color 0 0 0 0)
-	)
 	(no_connect
 		(at 21.59 107.95)
@@
 	(wire
 		(pts
-			(xy 35.56 35.56) (xy 36.83 35.56)
-		)
-		(stroke
-			(width 0)
-			(type default)
-		)
-	)
-	(wire
-		(pts
 			(xy 222.25 54.61) (xy 234.95 54.61)
 		)
@@
 	(wire
 		(pts
-			(xy 45.72 35.56) (xy 48.26 35.56)
+			(xy 45.72 35.56) (xy 46.99 35.56)
 		)
 		(stroke
@@
 	(wire
 		(pts
-			(xy 36.83 35.56) (xy 38.1 35.56)
+			(xy 35.56 35.56) (xy 38.1 35.56)
 		)
 		(stroke
@@
 	(wire
 		(pts
+			(xy 46.99 35.56) (xy 48.26 35.56)
+		)
+		(stroke
+			(width 0)
+			(type default)
+		)
+	)
+	(wire
+		(pts
 			(xy 69.85 69.85) (xy 71.12 69.85)
 		)
@@
 	(symbol
 		(lib_id "power:PWR_FLAG")
-		(at 36.83 35.56 0)
+		(at 46.99 35.56 0)
 		(unit 1)
 		(exclude_from_sim no)
@@
 		(dnp no)
 		(property "Reference" "#FLG01"
-			(at 36.83 33.655 0)
+			(at 46.99 33.655 0)
 			(effects
 				(font
@@
 		)
 		(property "Value" "PWR_FLAG"
-			(at 36.83 27.94 0)
+			(at 46.99 27.94 90)
 			(effects
 				(font
@@
 		)
 		(property "Footprint" ""
-			(at 36.83 35.56 0)
+			(at 46.99 35.56 0)
 			(effects
 				(font
@@
 		)
 		(property "Datasheet" "~"
-			(at 36.83 35.56 0)
+			(at 46.99 35.56 0)
 			(effects
 				(font
@@
 		)
 		(property "Description" "Special symbol for telling ERC where power comes from"
-			(at 36.83 35.56 0)
+			(at 46.99 35.56 0)
 			(effects
 				(font

Commit message: Début routage
déput placement des composants sur pcb, et capa de decouplage relativement aux composants
Parts:
- H1, H2, H3, H4: footprint MountingHole:MountingHole_3.2mm_M3_DIN965 -> MountingHole:MountingHole_3.2mm_M3_DIN965_Pad_TopBottom
- U1: footprint ESP32_DEVKITC_32UE:ESPRESSIF_ESP32-DEVKITC-32UE -> footprints:ESPRESSIF_ESP32-DEVKITC-32UE
- U2, U3: footprint (none) -> footprints:SSOP5_ROM-L
- U5: footprint (none) -> footprints:VQFN-HR_RYA_TEX
Other:
- note added: "23/09/2025"
