File: PCB/PCBs_v2/Partie_cmd/Partie_cmd.kicad_sch (KiCad schematic)
At the start: 0 parts

Commit message: Création du pcb cmd
Parts:
- added C3: 470u, Capacitor_SMD:C_0603_1608Metric_Pad1.08x0.95mm_HandSolder, symbol Device:C_Polarized_Small
- added C5, C9: 1u, Capacitor_SMD:C_0603_1608Metric_Pad1.08x0.95mm_HandSolder, symbol Device:C_Small
- added C6: 105n, Capacitor_SMD:C_0603_1608Metric_Pad1.08x0.95mm_HandSolder, symbol Device:C_Small
- added C7: 180u, Capacitor_SMD:C_0603_1608Metric_Pad1.08x0.95mm_HandSolder, symbol Device:C_Polarized_Small
- added D10, D11, D3, D4, D5, D8, D9: LED_Small, LED_SMD:LED_0603_1608Metric_Pad1.05x0.95mm_HandSolder, symbol Device:LED_Small
- added D2: MBRS320, Diode_SMD:D_SMC, symbol Diode:1N5820
- added J1: Barrel_Jack, symbol Connector:Barrel_Jack
- added J2, J3: Conn_01x04_Socket, Connector_PinSocket_1.27mm:PinSocket_1x04_P1.27mm_Vertical, symbol Connector:Conn_01x04_Socket
- added J4: Conn_01x11_Pin, symbol Connector:Conn_01x11_Pin
- added J5: Conn_01x10_Pin, symbol Connector:Conn_01x10_Pin
- added JP_tp_12V, JP_tp_3v3, JP_tp_5V, JP_tp_AIN1, JP_tp_AIN2, JP_tp_BIN1, JP_tp_BIN2, JP_tp_FSYNC, JP_tp_IRQZ, JP_tp_PWMA, JP_tp_PWMB, JP_tp_SBCLK, JP_tp_SCL, JP_tp_SDA, JP_tp_SDIN, JP_tp_SDOUT, JP_tp_SDZ, JP_tp_STBY, JP_tp_echo_cap_1, JP_tp_echo_cap_2, JP_tp_trig_cap_1, JP_tp_trig_cap_2: SolderJumper_2_Open, Jumper:SolderJumper-2_P1.3mm_Open_TrianglePad1.0x1.5mm, symbol Jumper:SolderJumper_2_Open
- added L1: 68u, Inductor_SMD:L_0805_2012Metric_Pad1.05x1.20mm_HandSolder, symbol Device:L_Small
- added R1: 4,7k, Resistor_SMD:R_0603_1608Metric_Pad0.98x0.95mm_HandSolder, symbol Device:R_Small
- added R2, R3, R4, R6, R7: 120, Resistor_SMD:R_0603_1608Metric_Pad0.98x0.95mm_HandSolder, symbol Device:R_Small
- added R5: 82, Resistor_SMD:R_0603_1608Metric_Pad0.98x0.95mm_HandSolder, symbol Device:R_Small
- added SW1: SW_MEC_5G, symbol Switch:SW_MEC_5G
- added U1: ESP32-S3-DEVKITC-1-N8R2, ESP32-S3-DEVKITC-1-N8R2:XCVR_ESP32-S3-DEVKITC-1-N8R2, symbol ESP32-S3-DEVKITC-1-N8R2:ESP32-S3-DEVKITC-1-N8R2
- added U3: BU33SD5WG-TR, footprints:SSOP5_ROM-L, symbol 2025-09-19_12-39-26:BU33SD5WG-TR
- added U4: XL1509-5.0, Package_SO:SOIC-8_3.9x4.9mm_P1.27mm, symbol Regulator_Switching:XL1509-5.0
Connections:
- new net: J1.1, SW1.1 (A), SW1.2 (A)
- new net: D4.2 (A), R4.2
- new net: D3.2 (A), R1.2
- new net: JP_tp_SDZ.2 (B), U1.J1_10 (GPIO17)
- new net: R7.1, U1.J3_12 (GPIO36)
- new net: D11.2 (A), R7.2
- new net: C9.1, JP_tp_3v3.1 (A), U3.5 (VOUT)
- new net: C7.1, JP_tp_5V.1 (A), L1.2, U4.3 (FB)
- new net: JP_tp_IRQZ.2 (B), U1.J1_11 (GPIO18)
- new net: JP_tp_PWMA.2 (B), U1.J1_12 (GPIO8)
- new net: JP_tp_echo_cap_2.2 (B), U1.J1_13 (GPIO3)
- new net: JP_tp_PWMB.2 (B), U1.J1_15 (GPIO9)
- new net: JP_tp_SDA.2 (B), U1.J1_16 (GPIO10)
- new net: JP_tp_SCL.2 (B), U1.J1_17 (GPIO11)
- new net: JP_tp_SDOUT.2 (B), U1.J1_18 (GPIO12)
- new net: JP_tp_SDIN.2 (B), U1.J1_19 (GPIO13)
- new net: JP_tp_SBCLK.2 (B), U1.J1_20 (GPIO14)
- new net: JP_tp_AIN1.2 (B), U1.J1_4 (GPIO4)
- new net: JP_tp_AIN2.2 (B), U1.J1_5 (GPIO5)
- new net: JP_tp_BIN1.2 (B), U1.J1_6 (GPIO6)
- new net: JP_tp_BIN2.2 (B), U1.J1_7 (GPIO7)
- new net: JP_tp_FSYNC.2 (B), U1.J1_8 (GPIO15)
- new net: JP_tp_STBY.2 (B), U1.J1_9 (GPIO16)
- new net: R3.1, U1.J3_10 (GPIO38)
- new net: R6.1, U1.J3_11 (GPIO37)
- new net: JP_tp_trig_cap_1.2 (B), U1.J3_14 (GPIO0)
- new net: JP_tp_echo_cap_1.2 (B), U1.J3_4 (GPIO1)
- new net: JP_tp_trig_cap_2.2 (B), U1.J3_5 (GPIO2)
- new net: R2.1, U1.J3_9 (MTCK/GPIO39)
- new net: D2.1 (K), L1.1, U4.2 (OUT)
- new net: D8.2 (A), R2.2
- new net: D10.2 (A), R6.2
- new net: JP_tp_12V.1 (A), SW1.3 (B), SW1.4 (B)
- new net: D9.2 (A), R3.2
- new net: D5.2 (A), R5.2
- new net 1.8V: J4.2 (Pin_2), R5.1
- new net 12V: C3.1, C6.1, J4.1 (Pin_1), J5.1 (Pin_1), JP_tp_12V.2 (B), R1.1, U4.1 (VIN)
- new net 3.3V: J5.2 (Pin_2), JP_tp_3v3.2 (B), R4.1, U1.J1_1 (3V3), U1.J1_2 (3V3__1)
- new net 5V: C5.1, J2.1 (Pin_1), J3.1 (Pin_1), JP_tp_5V.2 (B), U1.J1_21 (5V0), U3.1 (VIN), U3.3 (STBY)
- new net AIN1: J5.7 (Pin_7), JP_tp_AIN1.1 (A)
- new net AIN2: J5.8 (Pin_8), JP_tp_AIN2.1 (A)
- new net BIN1: J5.9 (Pin_9), JP_tp_BIN1.1 (A)
- new net BIN2: J5.10 (Pin_10), JP_tp_BIN2.1 (A)
- new net Echo_cap_1: J3.3 (Pin_3), JP_tp_echo_cap_1.1 (A)
- new net Echo_cap_2: J2.3 (Pin_3), JP_tp_echo_cap_2.1 (A)
- new net FSYNC: J4.5 (Pin_5), JP_tp_FSYNC.1 (A)
- new net GND: C3.2, C5.2, C6.2, C7.2, C9.2, D10.1 (K), D11.1 (K), D2.2 (A), D3.1 (K), D4.1 (K), D5.1 (K), D8.1 (K), D9.1 (K), J1.2, J2.4 (Pin_4), J3.4 (Pin_4), J4.3 (Pin_3), J5.3 (Pin_3), U1.J1_22 (GND), U1.J3_1 (GND__1), U1.J3_21 (GND__2), U1.J3_22 (GND__3), U3.2 (GND), U4.4 (~{EN}), U4.5 (GND), U4.6 (GND), U4.7 (GND), U4.8 (GND)
- new net IRQZ: J4.9 (Pin_9), JP_tp_IRQZ.1 (A)
- new net PWMA: J5.5 (Pin_5), JP_tp_PWMA.1 (A)
- new net PWMB: J5.6 (Pin_6), JP_tp_PWMB.1 (A)
- new net SBCLK: J4.4 (Pin_4), JP_tp_SBCLK.1 (A)
- new net SCL: J4.11 (Pin_11), JP_tp_SCL.1 (A)
- new net SDA: J4.10 (Pin_10), JP_tp_SDA.1 (A)
- new net SDIN: J4.6 (Pin_6), JP_tp_SDIN.1 (A)
- new net SDOUT: J4.7 (Pin_7), JP_tp_SDOUT.1 (A)
- new net SDZ: J4.8 (Pin_8), JP_tp_SDZ.1 (A)
- new net STBY: J5.4 (Pin_4), JP_tp_STBY.1 (A)
- new net Trig_cap_1: J3.2 (Pin_2), JP_tp_trig_cap_1.1 (A)
- new net Trig_cap_2: J2.2 (Pin_2), JP_tp_trig_cap_2.1 (A)
- no-connect marks 0 -> 14
Other:
- note added: "Conn carte drivers"
- note added: "Conn carte moteur"
