File: PCB/PCBs_v2/Partie_cmd/Partie_cmd.kicad_pcb (KiCad board)
At the start: 4 copper layers, 79.2 x 75 mm, 74 parts, among them J1 Barrel_Jack, J10 Conn_01x02, J2 Conn_01x04_Socket, J3 Conn_01x04_Socket, J5 Conn_01x14, J6 Conn_01x04, J7 Conn_01x04, J9 Conn_01x02, U1 ESP32-S3-DEVKITC-1-N8R2, U2 BU18SD5WG-TL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

Commit message: correction erreurs
Routing:
- net GND: track 106.4 -> 114.4 mm, vias 31 -> 79
- net Echo_cap_2: track 52.8 -> 54.6 mm
- net 5V: track 238.3 -> 238.8 mm
