File: PCB/PCB_v1/Nomad.kicad_sch (KiCad schematic)
At the start: 61 parts, among them J1 Barrel_Jack, J2 Conn_01x04_Socket, J3 Conn_01x04_Socket, J4 Conn_01x02_Socket, J5 Conn_01x02_Socket, U2 BU18SD5WG-TL, U3 BU33SD5WG-TR, U4 XL1509-5.0, U5 PTAS2780RYAR, U6 ESP32-S3-DEVKITC-1-N8R2

Commit message: Routage pcb cmd
Changed lines of the file:
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@@
-	(wire
-		(pts
-			(xy 138.43 185.42) (xy 140.97 185.42)
-		)
-		(stroke
-			(width 0)
-			(type default)
-		)
-	)
 	(wire
 		(pts
@@
 	(wire
 		(pts
-			(xy 143.51 184.15) (xy 143.51 185.42)
-		)
-		(stroke
-			(width 0)
-			(type default)
-		)
-	)
-	(wire
-		(pts
 			(xy 46.99 34.29) (xy 46.99 35.56)
 		)
@@
 	(wire
 		(pts
+			(xy 140.97 185.42) (xy 138.43 185.42)
+		)
+		(stroke
+			(width 0)
+			(type default)
+		)
+	)
+	(wire
+		(pts
 			(xy 223.52 95.25) (xy 226.06 95.25)
 		)
@@
 	(wire
 		(pts
-			(xy 138.43 184.15) (xy 138.43 185.42)
-		)
-		(stroke
-			(width 0)
-			(type default)
-		)
-	)
-	(wire
-		(pts
 			(xy 72.39 41.91) (xy 72.39 43.18)
 		)
@@
 	(wire
 		(pts
+			(xy 143.51 185.42) (xy 143.51 184.15)
+		)
+		(stroke
+			(width 0)
+			(type default)
+		)
+	)
+	(wire
+		(pts
 			(xy 228.6 39.37) (xy 228.6 41.91)
 		)
@@
 		)
 		(stroke
+			(width 0)
+			(type default)
+		)
+	)
+	(wire
+		(pts
+			(xy 138.43 185.42) (xy 138.43 184.15)
+		)
+		(stroke
