File: PCB/PCBs_v2/Partie_audio/Audio.kicad_sch (KiCad schematic)
At the start: 24 parts, among them J1 Conn_01x11, J2 Conn_01x02, U1 PTAS2780RYAR

Commit message: MAJ PCB audio
Parts:
- removed J1: Conn_01x11, Connector_PinHeader_2.00mm:PinHeader_1x11_P2.00mm_Vertical, symbol Connector_Generic:Conn_01x11
- added J1: Conn_01x13, Connector_PinHeader_2.00mm:PinHeader_1x13_P2.00mm_Vertical, symbol Connector_Generic:Conn_01x13
Connections:
- net +1.8V: now also J1.9 (Pin_9)
- net +12V: now also J1.11 (Pin_11)
- net +5V: now also J1.10 (Pin_10)
- net FSYNC: now also J1.1 (Pin_1)
- net GND: now also J1.12 (Pin_12), J1.13 (Pin_13)
- net IRQZ: now also J1.7 (Pin_7)
- net SBCLK: now also J1.2 (Pin_2)
- net SCL: now also J1.4 (Pin_4)
- net SDA: now also J1.5 (Pin_5)
- net SDIN: now also J1.3 (Pin_3)
- net SDOUT: now also J1.8 (Pin_8)
- net SDZ: now also J1.6 (Pin_6)
Changed lines of the file:
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@@
 	(rectangle
 		(start 12.7 67.31)
-		(end 52.07 109.22)
+		(end 52.07 121.92)
 		(stroke
 			(width 0)
@@
 	)
 	(junction
+		(at 26.67 105.41)
+		(diameter 0)
+		(color 0 0 0 0)
+	)
+	(junction
 		(at 121.92 102.87)
 		(diameter 0)
@@
 	(wire
 		(pts
+			(xy 24.13 105.41) (xy 26.67 105.41)
+		)
+		(stroke
+			(width 0)
+			(type default)
+		)
+	)
+	(wire
+		(pts
 			(xy 24.13 100.33) (xy 30.48 100.33)
 		)
@@
 	(wire
 		(pts
+			(xy 24.13 102.87) (xy 26.67 102.87)
+		)
+		(stroke
+			(width 0)
+			(type default)
+		)
+	)
+	(wire
+		(pts
 			(xy 86.36 88.9) (xy 97.79 88.9)
 		)
@@
 	(wire
 		(pts
+			(xy 26.67 102.87) (xy 26.67 105.41)
+		)
+		(stroke
+			(width 0)
+			(type default)
+		)
+	)
+	(wire
+		(pts
 			(xy 186.69 45.72) (xy 187.96 45.72)
 		)
@@
 	(wire
 		(pts
+			(xy 26.67 105.41) (xy 30.48 105.41)
+		)
+		(stroke
+			(width 0)
+			(type default)
+		)
+	)
+	(wire
+		(pts
 			(xy 194.31 63.5) (xy 199.39 63.5)
 		)
@@
 	)
 	(symbol
-		(lib_id "Connector_Generic:Conn_01x11")
-		(at 19.05 87.63 0)
-		(mirror y)
-		(unit 1)
-		(exclude_from_sim no)
-		(in_bom yes)
-		(on_board yes)
-		(dnp no)
-		(property "Reference" "J1"
-			(at 19.05 103.886 0)
-			(effects
-				(font
-					(size 1.27 1.27)
-				)
-			)
-		)
-		(property "Value" "Conn_01x11"
-			(at 19.558 106.68 0)
-			(effects
-				(font
-					(size 1.27 1.27)
-				)
-			)
-		)
-		(property "Footprint" "Connector_PinHeader_2.00mm:PinHeader_1x11_P2.00mm_Vertical"
-			(at 19.05 87.63 0)
-			(effects
-				(font
-					(size 1.27 1.27)
-				)
-				(hide yes)
-			)
-		)
-		(property "Datasheet" "~"
-			(at 19.05 87.63 0)
-			(effects
-				(font
-					(size 1.27 1.27)
-				)
-				(hide yes)
-			)
-		)
-		(property "Description" "Generic connector, single row, 01x11, script generated (kicad-library-utils/schlib/autogen/connector/)"
-			(at 19.05 87.63 0)
-			(effects
-				(font
-					(size 1.27 1.27)
-				)
-				(hide yes)
-			)
-		)
-		(pin "9"
-		)
-		(pin "7"
-		)
-		(pin "5"
-		)
-		(pin "4"
-		)
-		(pin "8"
-		)
-		(pin "6"
-		)
-		(pin "1"
-		)
-		(pin "10"
-		)
-		(pin "3"
-		)
-		(pin "2"
-		)
-		(pin "11"
-		)
-		(instances
-			(project ""
-				(path "/f27d1d9c-39f2-458b-9d29-7532dd02c1a6"
-					(reference "J1")
-					(unit 1)
-				)
-			)
-		)
-	)
-	(symbol
 		(lib_id "TAS2780:PTAS2780RYAR")
 		(at 212.09 22.86 0)
@@
 	(symbol
 		(lib_id "power:GND")
+		(at 30.48 105.41 0)
+		(unit 1)
+		(exclude_from_sim no)
+		(in_bom yes)
+		(on_board yes)
+		(dnp no)
+		(fields_autoplaced yes)
+		(property "Reference" "#PWR015"
+			(at 30.48 111.76 0)
+			(effects
+				(font
+					(size 1.27 1.27)
+				)
+				(hide yes)
+			)
+		)
+		(property "Value" "GND"
+			(at 30.48 110.49 0)
+			(effects
+				(font
+					(size 1.27 1.27)
+				)
+			)
+		)
+		(property "Footprint" ""
+			(at 30.48 105.41 0)
+			(effects
+				(font
+					(size 1.27 1.27)
+				)
+				(hide yes)
+			)
+		)
+		(property "Datasheet" ""
+			(at 30.48 105.41 0)
+			(effects
+				(font
+					(size 1.27 1.27)
+				)
+				(hide yes)
+			)
+		)
+		(property "Description" "Power symbol creates a global label with name \"GND\" , ground"
+			(at 30.48 105.41 0)
+			(effects
+				(font
+					(size 1.27 1.27)
+				)
+				(hide yes)
+			)
+		)
+		(pin "1"
+		)
+		(instances
+			(project ""
+				(path "/f27d1d9c-39f2-458b-9d29-7532dd02c1a6"
+					(reference "#PWR015")
+					(unit 1)
+				)
+			)
+		)
+	)
+	(symbol
+		(lib_id "power:GND")
 		(at 186.69 46.99 0)
 		(unit 1)
@@
 					(unit 1)
 				)
+			)
+		)
+	)
+	(symbol
+		(lib_id "Connector_Generic:Conn_01x13")
+		(at 19.05 90.17 0)
+		(mirror y)
+		(unit 1)
+		(exclude_from_sim no)
+		(in_bom yes)
+		(on_board yes)
+		(dnp no)
+		(property "Reference" "J1"
+			(at 18.796 71.882 0)
+			(effects
+				(font
+					(size 1.27 1.27)
+				)
+			)
+		)
+		(property "Value" "Conn_01x13"
+			(at 20.574 110.998 0)
+			(effects
+				(font
+					(size 1.27 1.27)
+				)
+			)
+		)
+		(property "Footprint" "Connector_PinHeader_2.00mm:PinHeader_1x13_P2.00mm_Vertical"
+			(at 19.05 90.17 0)
+			(effects
+				(font
+					(size 1.27 1.27)
+				)
+				(hide yes)
+			)
+		)
+		(property "Datasheet" "~"
+			(at 19.05 90.17 0)
+			(effects
+				(font
+					(size 1.27 1.27)
+				)
+				(hide yes)
+			)
+		)
+		(property "Description" "Generic connector, single row, 01x13, script generated (kicad-library-utils/schlib/autogen/connector/)"
+			(at 19.05 90.17 0)
+			(effects
+				(font
+					(size 1.27 1.27)
+				)
+				(hide yes)
+			)
+		)
+		(pin "10"
+		)
+		(pin "2"
+		)
+		(pin "1"
+		)
+		(pin "3"
+		)
+		(pin "9"
+		)
+		(pin "11"
+		)
+		(pin "12"
+		)
+		(pin "4"
+		)
+		(pin "7"
+		)
+		(pin "6"
+		)
+		(pin "5"
+		)
+		(pin "13"
+		)
+		(pin "8"
+		)
+		(instances
+			(project ""
+				(path "/f27d1d9c-39f2-458b-9d29-7532dd02c1a6"
+					(reference "J1")
+					(unit 1)
+				)

Commit message: Modification du schéma et du routage de la partie audio
Parts:
- removed H3: MountingHole_Pad, MountingHole:MountingHole_2.2mm_M2_DIN965_Pad, symbol Mechanical:MountingHole_Pad
- removed J1: Conn_01x13, Connector_PinHeader_2.00mm:PinHeader_1x13_P2.00mm_Vertical, symbol Connector_Generic:Conn_01x13
- added J1: Conn_01x12, Connector_PinHeader_2.00mm:PinHeader_1x12_P2.00mm_Vertical, symbol Connector_Generic:Conn_01x12
- added R5: 0, Resistor_SMD:R_0603_1608Metric_Pad0.98x0.95mm_HandSolder, symbol Device:R_Small
Connections:
- net VSNSN_ is gone; now on net VSNSN: R1.2, U1.1 (VSNSN)
- net VSNSP_ is gone; now on net VSNSP: R2.2, U1.5 (VSNSP)
- net FSYNC: now also J1.7 (Pin_7)
- net GND: now also J1.11 (Pin_11)
- net IRQZ: now also J1.2 (Pin_2)
- net SBCLK: now also J1.6 (Pin_6)
- net SCL: now also J1.5 (Pin_5)
- net SDA: now also J1.4 (Pin_4)
- net SDIN: now also J1.8 (Pin_8)
- net SDOUT: now also J1.9 (Pin_9)
- net SDZ: now also J1.1 (Pin_1)
- net VSNSN: no longer C2.1, FB2.2, J2.2 (Pin_2), R1.1
- net VSNSP: no longer C1.2, FB1.2, J2.1 (Pin_1), R2.1
- net +1.8V renamed IOVDD
- net IOVDD: now also J1.3 (Pin_3), R5.1; no longer C9.1, U1.24 (AVDD)
- net +12V renamed PVDD
- net PVDD: now also J1.12 (Pin_12)
- net +5V renamed VBAT1S
- net VBAT1S: now also J1.10 (Pin_10)
- new net AVDD: C9.1, R5.2, U1.24 (AVDD)
- new net HP_N: C2.1, FB2.2, J2.2 (Pin_2), R1.1
- new net HP_P: C1.2, FB1.2, J2.1 (Pin_1), R2.1

Commit message: Modification du PCB audio pour avoir un connecteur de 14 broches
Parts:
- removed J1: Conn_01x12, Connector_PinHeader_2.00mm:PinHeader_1x12_P2.00mm_Vertical, symbol Connector_Generic:Conn_01x12
- added J1: Conn_01x14, Connector_PinHeader_2.00mm:PinHeader_1x14_P2.00mm_Vertical, symbol Connector_Generic:Conn_01x14
Connections:
- net GNDPWR is gone; now on net GND: U1.2 (PGND)
- net FSYNC: now also J1.7 (Pin_7)
- net GND: now also J1.11 (Pin_11), J1.12 (Pin_12)
- net IOVDD: now also J1.3 (Pin_3)
- net IRQZ: now also J1.2 (Pin_2)
- net PVDD: now also J1.13 (Pin_13), J1.14 (Pin_14)
- net SBCLK: now also J1.6 (Pin_6)
- net SCL: now also J1.5 (Pin_5)
- net SDA: now also J1.4 (Pin_4)
- net SDIN: now also J1.8 (Pin_8)
- net SDOUT: now also J1.9 (Pin_9)
- net SDZ: now also J1.1 (Pin_1)
- net VBAT1S: now also J1.10 (Pin_10)
