File: PCBs/Audio/Audio.kicad_sch (KiCad schematic)
At the start: 23 parts, among them J1 Conn_01x15, J2 Conn_01x02, U1 PTAS2780RYAR

Commit message: Modification du PCB de la partie audio pour avoir une perle de ferrite avec une ampreinte plus grande
Parts:
- FB1, FB2: footprint Capacitor_SMD:C_0805_2012Metric_Pad1.18x1.45mm_HandSolder -> Capacitor_SMD:C_1206_3216Metric_Pad1.33x1.80mm_HandSolder
Changed lines of the file:
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@@
 			)
 		)
-		(property "Footprint" "Capacitor_SMD:C_0805_2012Metric_Pad1.18x1.45mm_HandSolder"
+		(property "Footprint" "Capacitor_SMD:C_1206_3216Metric_Pad1.33x1.80mm_HandSolder"
 			(at 73.66 93.472 90)
 			(effects
@@
 			)
 		)
-		(property "Footprint" "Capacitor_SMD:C_0805_2012Metric_Pad1.18x1.45mm_HandSolder"
+		(property "Footprint" "Capacitor_SMD:C_1206_3216Metric_Pad1.33x1.80mm_HandSolder"
 			(at 73.66 86.868 90)
 			(effects
