File: PCBs/Commande/Partie_cmd.kicad_sch (KiCad schematic)
At the start: 74 parts, among them J1 Barrel_Jack, J10 Conn_01x02, J2 Conn_01x04_Socket, J3 Conn_01x04_Socket, J4 Conn_01x15, J6 Conn_01x04, J7 Conn_01x04, J9 Conn_01x02, U1 ESP32-S3-DEVKITC-1-N8R2, U2 BU18SD5WG-TL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

Commit message: Commande_Julie
Parts:
- J4: footprint Connector_PinSocket_1.27mm:PinSocket_1x15_P1.27mm_Vertical -> Connector_PinSocket_2.00mm:PinSocket_1x15_P2.00mm_Vertical
Changed lines of the file:
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@@
 	)
 	(junction
+		(at 57.15 170.18)
+		(diameter 0)
+		(color 0 0 0 0)
+	)
+	(junction
 		(at 193.04 38.1)
 		(diameter 0)
@@
 	(wire
 		(pts
+			(xy 57.15 170.18) (xy 58.42 170.18)
+		)
+		(stroke
+			(width 0)
+			(type default)
+		)
+	)
+	(wire
+		(pts
 			(xy 152.4 123.19) (xy 162.56 123.19)
 		)
@@
 	(wire
 		(pts
+			(xy 57.15 173.99) (xy 57.15 170.18)
+		)
+		(stroke
+			(width 0)
+			(type default)
+		)
+	)
+	(wire
+		(pts
 			(xy 118.11 120.65) (xy 127 120.65)
 		)
@@
 	(wire
 		(pts
+			(xy 55.88 170.18) (xy 55.88 166.37)
+		)
+		(stroke
+			(width 0)
+			(type default)
+		)
+	)
+	(wire
+		(pts
 			(xy 212.09 50.8) (xy 210.82 50.8)
 		)
@@
 	(wire
 		(pts
+			(xy 58.42 170.18) (xy 58.42 166.37)
+		)
+		(stroke
+			(width 0)
+			(type default)
+		)
+	)
+	(wire
+		(pts
 			(xy 33.02 102.87) (xy 26.67 102.87)
 		)
@@
 	(wire
 		(pts
+			(xy 57.15 170.18) (xy 55.88 170.18)
+		)
+		(stroke
+			(width 0)
+			(type default)
+		)
+	)
+	(wire
+		(pts
 			(xy 137.16 83.82) (xy 138.43 83.82)
 		)
@@
 	(symbol
 		(lib_id "power:GND")
-		(at 55.88 166.37 0)
+		(at 57.15 173.99 0)
 		(unit 1)
 		(exclude_from_sim no)
@@
 		(dnp no)
 		(property "Reference" "#PWR022"
-			(at 55.88 172.72 0)
+			(at 57.15 180.34 0)
 			(effects
 				(font
@@
 		)
 		(property "Value" "GND"
-			(at 54.102 169.926 0)
+			(at 55.118 180.594 0)
 			(effects
 				(font
@@
 		)
 		(property "Footprint" ""
-			(at 55.88 166.37 0)
+			(at 57.15 173.99 0)
 			(effects
 				(font
@@
 		)
 		(property "Datasheet" ""
-			(at 55.88 166.37 0)
+			(at 57.15 173.99 0)
 			(effects
 				(font
@@
 		)
 		(property "Description" "Power symbol creates a global label with name \"GND\" , ground"
-			(at 55.88 166.37 0)
+			(at 57.15 173.99 0)
 			(effects
 				(font
@@
 			)
 		)
-		(property "Footprint" "Connector_PinSocket_1.27mm:PinSocket_1x15_P1.27mm_Vertical"
+		(property "Footprint" "Connector_PinSocket_2.00mm:PinSocket_1x15_P2.00mm_Vertical"
 			(at 48.26 161.29 0)
 			(effects
@@
 					(unit 1)
 				)
-			)
-		)
-	)
-	(symbol
-		(lib_id "power:GND")
-		(at 58.42 166.37 0)
-		(unit 1)
-		(exclude_from_sim no)
-		(in_bom yes)
-		(on_board yes)
-		(dnp no)
-		(property "Reference" "#PWR024"
-			(at 58.42 172.72 0)
-			(effects
-				(font
-					(size 1.27 1.27)
-				)
-				(hide yes)
-			)
-		)
-		(property "Value" "GND"
-			(at 56.642 169.926 0)
-			(effects
-				(font
-					(size 1.27 1.27)
-				)
-				(justify left)
-			)
-		)
-		(property "Footprint" ""
-			(at 58.42 166.37 0)
-			(effects
-				(font
-					(size 1.27 1.27)
-				)
-				(hide yes)
-			)
-		)
-		(property "Datasheet" ""
-			(at 58.42 166.37 0)
-			(effects
-				(font
-					(size 1.27 1.27)
-				)
-				(hide yes)
-			)
-		)
-		(property "Description" "Power symbol creates a global label with name \"GND\" , ground"
-			(at 58.42 166.37 0)
-			(effects
-				(font
-					(size 1.27 1.27)
-				)
-				(hide yes)
-			)
-		)
-		(pin "1"
-		)
-		(instances
-			(project "Partie_cmd"
-				(path "/feb16e15-81d7-49b9-8315-2aeb60da597a"
-					(reference "#PWR024")
-					(unit 1)
-				)

Commit message: schema et pcb update
Parts:
- removed H5: MountingHole_Pad, MountingHole:MountingHole_2.2mm_M2_DIN965_Pad, symbol Mechanical:MountingHole_Pad
- removed J6: Conn_01x04, Connector_PinSocket_1.00mm:PinSocket_1x04_P1.00mm_Vertical, symbol Connector_Generic:Conn_01x04
- removed J7: Conn_01x04, Connector_PinHeader_1.27mm:PinHeader_1x04_P1.27mm_Vertical, symbol Connector_Generic:Conn_01x04
- added J5: Conn_01x08, Connector_PinHeader_2.54mm:PinHeader_1x08_P2.54mm_Vertical, symbol Connector_Generic:Conn_01x08
- added J8: Conn_01x06, Connector_PinHeader_2.54mm:PinHeader_1x06_P2.54mm_Vertical, symbol Connector_Generic:Conn_01x06
- C3: footprint Capacitor_SMD:C_0603_1608Metric_Pad1.08x0.95mm_HandSolder -> Capacitor_SMD:CP_Elec_8x10.5
- C7: value 180u -> 150u; footprint Capacitor_SMD:C_0603_1608Metric_Pad1.08x0.95mm_HandSolder -> Capacitor_SMD:CP_Elec_6.3x7.7
- H4: footprint MountingHole:MountingHole_2.2mm_M2_DIN965_Pad -> MountingHole:MountingHole_2.5mm_Pad_Via
- J2, J3: footprint Connector_PinSocket_1.27mm:PinSocket_1x04_P1.27mm_Vertical -> Connector_PinHeader_2.54mm:PinHeader_1x04_P2.54mm_Vertical
Connections:
- net 3.3V: now also J2.1 (Pin_1), J3.1 (Pin_1), R8.1, R9.1, J5.1 (Pin_1), J8.1 (Pin_1)
- net 5V: no longer J2.1 (Pin_1), J3.1 (Pin_1), R8.1, R9.1
- net GND: now also J5.2 (Pin_2), J8.2 (Pin_2)
- net SCL: now also J5.4 (Pin_4), J8.3 (Pin_3)
- net SDA: now also J5.3 (Pin_3), J8.4 (Pin_4)
- net at JP_tp_SDZ1.2 (B): now also U1.J1_11 (GPIO18); no longer U1.J1_10 (GPIO17)
- net at JP_tp_IRQZ1.2 (B): now also U1.J3_18 (GPIO21); no longer U1.J1_11 (GPIO18)
- net at U1.J1_12 (GPIO8): now also JP_tp_BIN2.2 (B); no longer JP_tp_PWMA1.2 (B)
- net at U1.J1_13 (GPIO3): now also JP_tp_trig_cap_2.2 (B); no longer JP_tp_echo_cap_2.2 (B)
- net at U1.J1_15 (GPIO9): now also JP_tp_PWMA1.2 (B); no longer JP_tp_PWMB1.2 (B)
- net at U1.J1_16 (GPIO10): now also JP_tp_PWMB1.2 (B); no longer JP_tp_SDA1.2 (B)
- net at U1.J1_17 (GPIO11): now also JP_tp_SDA1.2 (B); no longer JP_tp_SCL1.2 (B)
- net at U1.J1_18 (GPIO12): now also JP_tp_SCL1.2 (B); no longer JP_tp_SDOUT1.2 (B)
- net at U1.J1_19 (GPIO13): now also JP_tp_SDOUT1.2 (B); no longer JP_tp_SDIN1.2 (B)
- net at U1.J1_20 (GPIO14): now also JP_tp_SDIN1.2 (B); no longer JP_tp_SBCLK1.2 (B)
- net at U1.J1_4 (GPIO4): now also JP_tp_echo_cap_2.2 (B); no longer JP_tp_AIN1.2 (B)
- net at U1.J1_5 (GPIO5): now also JP_tp_AIN1.2 (B); no longer JP_tp_AIN2.2 (B)
- net at U1.J1_6 (GPIO6): now also JP_tp_AIN2.2 (B); no longer JP_tp_BIN1.2 (B)
- net at U1.J1_7 (GPIO7): now also JP_tp_BIN1.2 (B); no longer JP_tp_BIN2.2 (B)
- net at U1.J1_8 (GPIO15): now also JP_tp_SBCLK1.2 (B); no longer JP_tp_FSYNC1.2 (B)
- net at JP_tp_STBY1.2 (B): now also U1.J1_10 (GPIO17); no longer U1.J1_9 (GPIO16)
- net at U1.J3_14 (GPIO0): no longer JP_tp_trig_cap_1.2 (B)
- net at U1.J3_4 (GPIO1): now also JP_tp_trig_cap_1.2 (B); no longer JP_tp_echo_cap_1.2 (B)
- net at U1.J3_5 (GPIO2): now also JP_tp_echo_cap_1.2 (B); no longer JP_tp_trig_cap_2.2 (B)
- new net: JP_tp_FSYNC1.2 (B), U1.J1_9 (GPIO16)
- no-connect marks 14 -> 19
Other:
- moved on the sheet: C1, C10, C11, C2, C3, C4, C5, C6, C7, C8, C9, D1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

Commit message: pcbss
Parts:
- J1: footprint Connector_BarrelJack:BarrelJack_Wuerth_694108106102_2.5x5.5mm -> BarrelJack (PPZ):CONN3_06105102_WRE
Changed lines of the file:
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@@
 			)
 		)
-		(property "Footprint" "Connector_BarrelJack:BarrelJack_Wuerth_694108106102_2.5x5.5mm"
+		(property "Footprint" "BarrelJack (PPZ):CONN3_06105102_WRE"
 			(at 25.4 34.036 0)
 			(effects

Commit message: New pcb avec des erreurs
Parts:
- removed J1: Barrel_Jack, BarrelJack (PPZ):CONN3_06105102_WRE, symbol Connector:Barrel_Jack
- removed J10, J9: Conn_01x02, Connector_JST:JST_XH_B2B-XH-A_1x02_P2.50mm_Vertical, symbol Connector_Generic:Conn_01x02
- removed JP_tp_AIN1, JP_tp_AIN2, JP_tp_BIN1, JP_tp_BIN2, JP_tp_FSYNC1, JP_tp_IRQZ1, JP_tp_PWMA1, JP_tp_PWMB1, JP_tp_SBCLK1, JP_tp_SCL1, JP_tp_SDA1, JP_tp_SDIN1, JP_tp_SDOUT1, JP_tp_SDZ1, JP_tp_STBY1, JP_tp_echo_cap_1, JP_tp_echo_cap_2, JP_tp_trig_cap_1, JP_tp_trig_cap_2: SolderJumper_2_Open, Jumper:SolderJumper-2_P1.3mm_Open_TrianglePad1.0x1.5mm, symbol Jumper:SolderJumper_2_Open
- added J6: M1, Connector_JST:JST_PH_B6B-PH-K_1x06_P2.00mm_Vertical, symbol Connector_Generic:Conn_01x06
- added J7: M2, Connector_JST:JST_PH_B6B-PH-K_1x06_P2.00mm_Vertical, symbol Connector_Generic:Conn_01x06
- added J9: 694106105102, Jack (PPZ):CONN3_06105102_WRE, symbol Jack (PPZ):694106105102
- J2: value Conn_01x04_Socket -> UltraB
- J3: value Conn_01x04_Socket -> UltraF
- J4: value Conn_01x15 -> Audio
- J5: value Conn_01x08 -> Acc
- J8: value Conn_01x06 -> TOF
- renumbered JP_tp_12V1 to 12V1, JP_tp_1v8 to 1v8, JP_tp_3v3 to 3v3, JP_tp_5V1 to 5V1
Connections:
- net 5V: now also J6.5 (Pin_5), J7.5 (Pin_5)
- net AIN1: now also U1.J1_5 (GPIO5)
- net AIN2: now also U1.J1_6 (GPIO6)
- net AO1: now also J6.1 (Pin_1)
- net AO2: now also J6.6 (Pin_6)
- net BIN1: now also U1.J1_7 (GPIO7)
- net BIN2: now also U1.J1_12 (GPIO8)
- net BO1: now also J7.1 (Pin_1)
- net BO2: now also J7.6 (Pin_6)
- net Echo_cap_1: now also U1.J3_5 (GPIO2)
- net Echo_cap_2: now also U1.J1_4 (GPIO4)
- net FSYNC: now also U1.J1_9 (GPIO16)
- net GND: now also J6.2 (Pin_2), J7.2 (Pin_2), J9.2, J9.3
- net IRQZ: now also U1.J3_18 (GPIO21)
- net PWMA: now also U1.J1_15 (GPIO9)
- net PWMB: now also U1.J1_16 (GPIO10)
- net SBCLK: now also U1.J1_8 (GPIO15)
- net SCL: now also U1.J1_18 (GPIO12)
- net SDA: now also U1.J1_17 (GPIO11)
- net SDIN: now also U1.J1_20 (GPIO14)
- net SDOUT: now also U1.J1_19 (GPIO13)
- net SDZ: now also U1.J1_11 (GPIO18)
- net STBY: now also U1.J1_10 (GPIO17)
- net Trig_cap_1: now also U1.J3_4 (GPIO1)
- net Trig_cap_2: now also U1.J1_13 (GPIO3)
- net at JP1.1 (A): now also J9.1
- net C2A: now reaches U1.J3_16 (GPIO48)
- net C2A: now also J6.4 (Pin_4)
- net C1A: now reaches U1.J3_17 (GPIO47)
- net C1A: now also J6.3 (Pin_3)
- net C2B: now reaches U1.J3_19 (USB_D+/GPIO20)
- net C2B: now also J7.4 (Pin_4)
- net C1B: now reaches U1.J3_20 (USB_D-/GPIO19)
- net C1B: now also J7.3 (Pin_3)
- no-connect marks 19 -> 16
Other:
- note added: "Moteurs N20 encodeur"
- note removed: "Moteurs N20"
- moved on the sheet: 12V1, C1, C10, C11, C2, D1, D10, D11, D3, D4, D5, D6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

Commit message: edit pcb
Connections:
- net BIN1: now also U1.J1_16 (GPIO10); no longer U1.J1_7 (GPIO7)
- net BIN2: now also U1.J1_17 (GPIO11); no longer U1.J1_12 (GPIO8)
- net FSYNC: now also U1.J1_7 (GPIO7); no longer U1.J1_9 (GPIO16)
- net IRQZ: now also U1.J1_11 (GPIO18); no longer U1.J3_18 (GPIO21)
- net PWMA: now also U1.J1_12 (GPIO8); no longer U1.J1_15 (GPIO9)
- net PWMB: now also U1.J1_18 (GPIO12); no longer U1.J1_16 (GPIO10)
- net SCL: now also U1.J1_9 (GPIO16); no longer U1.J1_18 (GPIO12)
- net SDA: now also U1.J1_10 (GPIO17); no longer U1.J1_17 (GPIO11)
- net SDZ: now also U1.J3_18 (GPIO21); no longer U1.J1_11 (GPIO18)
- net STBY: now also U1.J1_15 (GPIO9); no longer U1.J1_10 (GPIO17)
Other:
- moved on the sheet: R8, R9

Commit message: Last pcbss
Parts:
- C6: value 105n -> 1u
Connections:
- net 1.8V: no longer J4.3 (Pin_3)
- net 3.3V: now also J4.3 (Pin_3); no longer J4.15 (Pin_15)
- no-connect marks 16 -> 17
Other:
- moved on the sheet: D5, D6, R10, R5
Changed lines of the file:
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@@
 	)
 	(no_connect
+		(at 181.61 124.46)
+	)
+	(no_connect
 		(at 189.23 77.47)
 	)
@@
 	(wire
 		(pts
-			(xy 66.04 157.48) (xy 67.31 157.48)
+			(xy 87.63 157.48) (xy 88.9 157.48)
 		)
 		(stroke
@@
 	(wire
 		(pts
-			(xy 93.98 157.48) (xy 92.71 157.48)
+			(xy 73.66 157.48) (xy 72.39 157.48)
 		)
 		(stroke
@@
 	(wire
 		(pts
-			(xy 73.66 158.75) (xy 73.66 157.48)
+			(xy 95.25 158.75) (xy 95.25 157.48)
 		)
 		(stroke
@@
 	(wire
 		(pts
-			(xy 86.36 157.48) (xy 87.63 157.48)
+			(xy 66.04 157.48) (xy 67.31 157.48)
 		)
 		(stroke
@@
 	(wire
 		(pts
-			(xy 93.98 158.75) (xy 93.98 157.48)
+			(xy 73.66 158.75) (xy 73.66 157.48)
 		)
 		(stroke
@@
 	(wire
 		(pts
-			(xy 73.66 163.83) (xy 73.66 165.1)
+			(xy 95.25 163.83) (xy 95.25 165.1)
 		)
 		(stroke
@@
 	(wire
 		(pts
-			(xy 93.98 163.83) (xy 93.98 165.1)
+			(xy 73.66 163.83) (xy 73.66 165.1)
 		)
 		(stroke
@@
 	(wire
 		(pts
-			(xy 73.66 157.48) (xy 72.39 157.48)
+			(xy 95.25 157.48) (xy 93.98 157.48)
 		)
 		(stroke
@@
 		)
 	)
-	(global_label "1.8V"
+	(global_label "3.3V"
 		(shape input)
 		(at 212.09 124.46 270)
@@
 		)
 	)
-	(global_label "3.3V"
-		(shape input)
-		(at 181.61 124.46 270)
-		(fields_autoplaced yes)
-		(effects
-			(font
-				(size 1.27 1.27)
-			)
-			(justify right)
-		)
-		(property "Intersheetrefs" "${INTERSHEET_REFS}"
-			(at 181.61 131.5576 90)
-			(effects
-				(font
-					(size 1.27 1.27)
-				)
-				(justify right)
-				(hide yes)
-			)
-		)
-	)
 	(global_label "BO1"
 		(shape input)
@@
 	(global_label "1.8V"
 		(shape input)
-		(at 66.04 157.48 180)
+		(at 87.63 157.48 180)
 		(fields_autoplaced yes)
 		(effects
@@
 		)
 		(property "Intersheetrefs" "${INTERSHEET_REFS}"
-			(at 58.9424 157.48 0)
+			(at 80.5324 157.48 0)
 			(effects
 				(font
@@
 	(global_label "3.3V"
 		(shape input)
-		(at 86.36 157.48 180)
+		(at 66.04 157.48 180)
 		(fields_autoplaced yes)
 		(effects
@@
 		)
 		(property "Intersheetrefs" "${INTERSHEET_REFS}"
-			(at 79.2624 157.48 0)
+			(at 58.9424 157.48 0)
 			(effects
 				(font
@@
 	(symbol
 		(lib_id "power:GND")
-		(at 73.66 165.1 0)
+		(at 95.25 165.1 0)
 		(unit 1)
 		(exclude_from_sim no)
@@
 		(fields_autoplaced yes)
 		(property "Reference" "#PWR019"
-			(at 73.66 171.45 0)
+			(at 95.25 171.45 0)
 			(effects
 				(font
@@
 		)
 		(property "Value" "GND"
-			(at 73.66 170.18 0)
+			(at 95.25 170.18 0)
 			(effects
 				(font
@@
 		)
 		(property "Footprint" ""
-			(at 73.66 165.1 0)
+			(at 95.25 165.1 0)
 			(effects
 				(font
@@
 		)
 		(property "Datasheet" ""
-			(at 73.66 165.1 0)
+			(at 95.25 165.1 0)
 			(effects
 				(font
@@
 		)
 		(property "Description" "Power symbol creates a global label with name \"GND\" , ground"
-			(at 73.66 165.1 0)
+			(at 95.25 165.1 0)
 			(effects
 				(font
@@
 	(symbol
 		(lib_id "power:GND")
-		(at 93.98 165.1 0)
+		(at 73.66 165.1 0)
 		(unit 1)
 		(exclude_from_sim no)
@@
 		(fields_autoplaced yes)
 		(property "Reference" "#PWR04"
-			(at 93.98 171.45 0)
+			(at 73.66 171.45 0)
 			(effects
 				(font
@@
 		)
 		(property "Value" "GND"
-			(at 93.98 170.18 0)
+			(at 73.66 170.18 0)
 			(effects
 				(font
@@
 		)
 		(property "Footprint" ""
-			(at 93.98 165.1 0)
+			(at 73.66 165.1 0)
 			(effects
 				(font
@@
 		)
 		(property "Datasheet" ""
-			(at 93.98 165.1 0)
+			(at 73.66 165.1 0)
 			(effects
 				(font
@@
 		)
 		(property "Description" "Power symbol creates a global label with name \"GND\" , ground"
-			(at 93.98 165.1 0)
+			(at 73.66 165.1 0)
 			(effects
 				(font
@@
 	(symbol
 		(lib_id "Device:R_Small")
-		(at 90.17 157.48 90)
+		(at 69.85 157.48 90)
 		(unit 1)
 		(exclude_from_sim no)
@@
 		(dnp no)
 		(property "Reference" "R10"
-			(at 83.82 151.13 90)
+			(at 63.5 151.13 90)
 			(effects
 				(font
@@
 		)
 		(property "Value" "1.2k"
-			(at 83.82 153.67 90)
+			(at 63.5 153.67 90)
 			(effects
 				(font
@@
 		)
 		(property "Footprint" "Resistor_SMD:R_0603_1608Metric_Pad0.98x0.95mm_HandSolder"
-			(at 90.17 157.48 0)
+			(at 69.85 157.48 0)
 			(effects
 				(font
@@
 		)
 		(property "Datasheet" "~"
-			(at 90.17 157.48 0)
+			(at 69.85 157.48 0)
 			(effects
 				(font
@@
 		)
 		(property "Description" "Resistor, small symbol"
-			(at 90.17 157.48 0)
+			(at 69.85 157.48 0)
 			(effects
 				(font
@@
 			)
 		)
-		(property "Value" "105n"
+		(property "Value" "1u"
 			(at 33.02 72.3962 0)
 			(effects
@@
 	(symbol
 		(lib_id "Device:LED_Small")
-		(at 73.66 161.29 270)
+		(at 95.25 161.29 270)
 		(mirror x)
 		(unit 1)
@@
 		(dnp no)
 		(property "Reference" "D5"
-			(at 71.12 162.56 90)
+			(at 92.71 162.56 90)
 			(effects
 				(font
@@
 		)
 		(property "Value" "LED_Small"
-			(at 71.12 162.4964 90)
+			(at 92.71 162.4964 90)
 			(effects
 				(font
@@
 		)
 		(property "Footprint" "LED_SMD:LED_0603_1608Metric_Pad1.05x0.95mm_HandSolder"
-			(at 73.66 161.29 90)
+			(at 95.25 161.29 90)
 			(effects
 				(font
@@
 		)
 		(property "Datasheet" "~"
-			(at 73.66 161.29 90)
+			(at 95.25 161.29 90)
 			(effects
 				(font
@@
 		)
 		(property "Description" "Light emitting diode, small symbol"
-			(at 73.66 161.29 0)
+			(at 95.25 161.29 0)
 			(effects
 				(font
@@
 		)
 		(property "Sim.Pin" "1=K 2=A"
-			(at 73.66 161.29 0)
+			(at 95.25 161.29 0)
 			(effects
 				(font
@@
 	(symbol
 		(lib_id "Device:LED_Small")
-		(at 93.98 161.29 270)
+		(at 73.66 161.29 270)
 		(mirror x)
 		(unit 1)
@@
 		(dnp no)
 		(property "Reference" "D6"
-			(at 92.202 162.052 90)
+			(at 71.882 162.052 90)
 			(effects
 				(font
@@
 		)
 		(property "Value" "LED_Small"
-			(at 91.44 162.4964 90)
+			(at 71.12 162.4964 90)
 			(effects
 				(font
@@
 		)
 		(property "Footprint" "LED_SMD:LED_0603_1608Metric_Pad1.05x0.95mm_HandSolder"
-			(at 93.98 161.29 90)
+			(at 73.66 161.29 90)
 			(effects
 				(font
@@
 		)
 		(property "Datasheet" "~"
-			(at 93.98 161.29 90)
+			(at 73.66 161.29 90)
 			(effects
 				(font
@@
 		)
 		(property "Description" "Light emitting diode, small symbol"
-			(at 93.98 161.29 0)
+			(at 73.66 161.29 0)
 			(effects
 				(font
@@
 		)
 		(property "Sim.Pin" "1=K 2=A"
-			(at 93.98 161.29 0)
+			(at 73.66 161.29 0)
 			(effects
 				(font
@@
 	(symbol
 		(lib_id "Device:R_Small")
-		(at 69.85 157.48 90)
+		(at 91.44 157.48 90)
 		(unit 1)
 		(exclude_from_sim no)
@@
 		(fields_autoplaced yes)
 		(property "Reference" "R5"
-			(at 69.85 152.4 90)
+			(at 91.44 152.4 90)
 			(effects
 				(font
@@
 		)
 		(property "Value" "820"
-			(at 69.85 154.94 90)
+			(at 91.44 154.94 90)
 			(effects
 				(font
@@
 		)
 		(property "Footprint" "Resistor_SMD:R_0603_1608Metric_Pad0.98x0.95mm_HandSolder"
-			(at 69.85 157.48 0)
+			(at 91.44 157.48 0)
 			(effects
 				(font
@@
 		)
 		(property "Datasheet" "~"
-			(at 69.85 157.48 0)
+			(at 91.44 157.48 0)
 			(effects
 				(font
@@
 		)
 		(property "Description" "Resistor, small symbol"
-			(at 69.85 157.48 0)
+			(at 91.44 157.48 0)
 			(effects
 				(font
